File: flight_computer/can_transceiver.kicad_sch (KiCad schematic)
At the start: 9 parts

Commit message: interconnect
Parts:
- renumbered C to C5, C to C6, D to D3, JP to JP4, R to R6, R to R7, U to U4
Other:
- note removed: "ESD Protection"
- note removed: "Optional Termination"
Changed lines of the file:
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@@
 		)
 	)
-	(text "ESD Protection\n"
+	(text_box "Optional Termination"
 		(exclude_from_sim no)
-		(at 194.818 145.288 0)
+		(at 142.24 83.82 0)
+		(size 29.21 63.5)
+		(margins 0.9525 0.9525 0.9525 0.9525)
+		(stroke
+			(width 0)
+			(type dash)
+			(color 0 0 194 1)
+		)
+		(fill
+			(type none)
+		)
 		(effects
 			(font
@@
 				(color 0 0 194 1)
 			)
-		)
-	)
-	(text "Optional Termination"
+			(justify right bottom)
+		)
+	)
+	(text_box "ESD Protection\n"
 		(exclude_from_sim no)
-		(at 160.274 145.288 0)
+		(at 173.99 83.82 0)
+		(size 29.21 63.5)
+		(margins 0.9525 0.9525 0.9525 0.9525)
+		(stroke
+			(width 0)
+			(type dash)
+			(color 0 0 194 1)
+		)
+		(fill
+			(type none)
+		)
 		(effects
 			(font
@@
 				(color 0 0 194 1)
 			)
+			(justify right bottom)
 		)
 	)
@@
 		(dnp no)
 		(fields_autoplaced yes)
-		(property "Reference" "C"
+		(property "Reference" "C5"
 			(at 121.92 66.04 90)
 			(show_name no)
@@
 			(project "flight_computer"
 				(path "/4b3676e8-35c3-4ec2-859c-99a6df767b3c/5251f0f1-b4ab-42e5-abc1-cd87dd350edb"
+					(reference "C5")
+					(unit 1)
+				)
+				(path "/4b3676e8-35c3-4ec2-859c-99a6df767b3c/adc3643f-6d6d-4902-b902-785309a5e75b"
 					(reference "C5")
 					(unit 1)
@@
 		(dnp no)
 		(fields_autoplaced yes)
-		(property "Reference" "#PWR"
+		(property "Reference" "#PWR07"
 			(at 129.54 83.82 0)
 			(hide yes)
@@
 			(project "flight_computer"
 				(path "/4b3676e8-35c3-4ec2-859c-99a6df767b3c/5251f0f1-b4ab-42e5-abc1-cd87dd350edb"
+					(reference "#PWR07")
+					(unit 1)
+				)
+				(path "/4b3676e8-35c3-4ec2-859c-99a6df767b3c/adc3643f-6d6d-4902-b902-785309a5e75b"
 					(reference "#PWR07")
 					(unit 1)
@@
 		(dnp no)
 		(fields_autoplaced yes)
-		(property "Reference" "R"
+		(property "Reference" "R7"
 			(at 153.67 115.5699 0)
 			(show_name no)
@@
 			(project "flight_computer"
 				(path "/4b3676e8-35c3-4ec2-859c-99a6df767b3c/5251f0f1-b4ab-42e5-abc1-cd87dd350edb"
+					(reference "R7")
+					(unit 1)
+				)
+				(path "/4b3676e8-35c3-4ec2-859c-99a6df767b3c/adc3643f-6d6d-4902-b902-785309a5e75b"
 					(reference "R7")
 					(unit 1)
@@
 		(dnp no)
 		(fields_autoplaced yes)
-		(property "Reference" "JP"
+		(property "Reference" "JP4"
 			(at 153.67 104.1399 90)
 			(show_name no)
@@
 			(project "flight_computer"
 				(path "/4b3676e8-35c3-4ec2-859c-99a6df767b3c/5251f0f1-b4ab-42e5-abc1-cd87dd350edb"
+					(reference "JP4")
+					(unit 1)
+				)
+				(path "/4b3676e8-35c3-4ec2-859c-99a6df767b3c/adc3643f-6d6d-4902-b902-785309a5e75b"
 					(reference "JP4")
 					(unit 1)
@@
 		(dnp no)
 		(fields_autoplaced yes)
-		(property "Reference" "C"
+		(property "Reference" "C6"
 			(at 160.02 126.9999 0)
 			(show_name no)
@@
 			(project "flight_computer"
 				(path "/4b3676e8-35c3-4ec2-859c-99a6df767b3c/5251f0f1-b4ab-42e5-abc1-cd87dd350edb"
+					(reference "C6")
+					(unit 1)
+				)
+				(path "/4b3676e8-35c3-4ec2-859c-99a6df767b3c/adc3643f-6d6d-4902-b902-785309a5e75b"
 					(reference "C6")
 					(unit 1)
@@
 		(dnp no)
 		(fields_autoplaced yes)
-		(property "Reference" "U"
+		(property "Reference" "U4"
 			(at 116.4433 102.87 0)
 			(show_name no)
@@
 			(project "flight_computer"
 				(path "/4b3676e8-35c3-4ec2-859c-99a6df767b3c/5251f0f1-b4ab-42e5-abc1-cd87dd350edb"
+					(reference "U4")
+					(unit 1)
+				)
+				(path "/4b3676e8-35c3-4ec2-859c-99a6df767b3c/adc3643f-6d6d-4902-b902-785309a5e75b"
 					(reference "U4")
 					(unit 1)
@@
 		(dnp no)
 		(fields_autoplaced yes)
-		(property "Reference" "R"
+		(property "Reference" "R6"
 			(at 95.25 78.7399 0)
 			(show_name no)
@@
 			(project "flight_computer"
 				(path "/4b3676e8-35c3-4ec2-859c-99a6df767b3c/5251f0f1-b4ab-42e5-abc1-cd87dd350edb"
+					(reference "R6")
+					(unit 1)
+				)
+				(path "/4b3676e8-35c3-4ec2-859c-99a6df767b3c/adc3643f-6d6d-4902-b902-785309a5e75b"
 					(reference "R6")
 					(unit 1)
@@
 		(dnp no)
 		(fields_autoplaced yes)
-		(property "Reference" "D"
+		(property "Reference" "D3"
 			(at 189.23 111.76 0)
 			(show_name no)
@@
 					(reference "D3")
 					(unit 1)
+				)
+				(path "/4b3676e8-35c3-4ec2-859c-99a6df767b3c/adc3643f-6d6d-4902-b902-785309a5e75b"
+					(reference "D3")
+					(unit 1)

Commit message: flight computer mcu
Parts:
- R6: value 100k -> 10k
Changed lines of the file:
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@@
 	(generator_version "10.0")
 	(paper "A4")
-	(rectangle
-		(start 142.24 83.82)
-		(end 171.45 147.32)
-		(stroke
-			(width 0)
-			(type dash)
-			(color 0 0 194 1)
-		)
-		(fill
-			(type none)
-		)
-	)
-	(rectangle
-		(start 173.99 83.82)
-		(end 203.2 147.32)
-		(stroke
-			(width 0)
-			(type dash)
-			(color 0 0 194 1)
-		)
-		(fill
-			(type none)
-		)
-	)
 	(text_box "Optional Termination"
 		(exclude_from_sim no)
-		(at 142.24 83.82 0)
-		(size 29.21 63.5)
+		(at 143.51 83.82 0)
+		(size 26.67 63.5)
 		(margins 0.9525 0.9525 0.9525 0.9525)
 		(stroke
@@
 	(text_box "ESD Protection\n"
 		(exclude_from_sim no)
-		(at 173.99 83.82 0)
+		(at 175.26 83.82 0)
 		(size 29.21 63.5)
+		(margins 0.9525 0.9525 0.9525 0.9525)
+		(stroke
+			(width 0)
+			(type dash)
+			(color 0 0 194 1)
+		)
+		(fill
+			(type none)
+		)
+		(effects
+			(font
+				(size 1.27 1.27)
+				(color 0 0 194 1)
+			)
+			(justify right bottom)
+		)
+	)
+	(text_box "CAN Transceiver"
+		(exclude_from_sim no)
+		(at 69.85 58.42 0)
+		(size 68.58 68.58)
 		(margins 0.9525 0.9525 0.9525 0.9525)
 		(stroke
@@
 			)
 		)
-		(property "Value" "100k"
+		(property "Value" "10k"
 			(at 95.25 81.2799 0)
 			(show_name no)
