File: flight_computer/interconnect.kicad_sch (KiCad schematic)
At the start: 16 parts, among them J1 DF12NB(5.0)-40DP-0.5V(51, J2 DF12NB-40DS-0.5V(51), U2 TPS255xxDBV, U3 TPS255xxDBV

Commit message: flight computer mcu
Parts:
- R1, R2, R4, R5: value 100k -> 4k7
- R11, R9: value 100k -> 10k
Changed lines of the file:
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@@
 			)
 		)
-		(property "Value" "100k"
+		(property "Value" "4k7"
 			(at 226.06 71.12 90)
 			(show_name no)
@@
 			)
 		)
-		(property "Value" "100k"
+		(property "Value" "10k"
 			(at 54.61 166.37 90)
 			(show_name no)
@@
 			)
 		)
-		(property "Value" "100k"
+		(property "Value" "4k7"
 			(at 226.06 44.45 90)
 			(show_name no)
@@
 			)
 		)
-		(property "Value" "100k"
+		(property "Value" "4k7"
 			(at 226.06 55.88 90)
 			(show_name no)
@@
 			)
 		)
-		(property "Value" "100k"
+		(property "Value" "10k"
 			(at 54.61 127 90)
 			(show_name no)
@@
 			)
 		)
-		(property "Value" "100k"
+		(property "Value" "4k7"
 			(at 226.06 82.55 90)
 			(show_name no)
