File: flight_computer/mcu.kicad_sch (KiCad schematic)
At the start: 5 parts, among them U1 STM32H563RGTx, Y1 MST8011xx-2x-xxE

Commit message: flight computer mcu
Parts:
- added C10, C11, C4, C7, C8, C9: 100n, symbol Device:C
- added C12: 1u, symbol Device:C
- added C13, C14, C16: 2u2, symbol Device:C
- added C15: 10n, symbol Device:C
- added C24: 100n, Capacitor_SMD:C_0402_1005Metric, symbol Device:C
- added D7: ESD5ZL5-1F4, Diode_SMD:D_0201_0603Metric, symbol Diode:ESD5Zxx
- added FB1: 74279265, Inductor_SMD:L_0603_1608Metric, symbol Device:FerriteBead
- added J3: DEBUG, symbol Connector_Generic_MountingPin:Conn_01x06_MountingPin
- added J4: Micro_SD_Card, Connector_Card:microSD_HC_Molex_47219-2001, symbol Connector:Micro_SD_Card
- added JP1: BOOT, symbol Jumper:SolderJumper_2_Open
- added R15, R16, R17, R18, R19: 10k, symbol Device:R
- added TP1: MCO, symbol Connector:TestPoint
- added U5: W25Q128JVS, Package_SO:SOIC-8_5.3x5.3mm_P1.27mm, symbol Memory_Flash:W25Q128JVS
- added U7: TPD6E05U06RVZ, Package_SON:Texas_R-PUSON-N14, symbol Power_Protection:TPD6E05U06RVZ
Connections:
- net 3V3 is gone; now on net VDD3V3: C3.1, R13.1, Y1.4 (VDD)
- net GND: now also U1.12 (VSSA), U1.18 (VSS), U1.31 (VSS), U1.47 (VSS), U1.63 (VSS), C10.2, C11.2, C12.2, C13.2, C14.2, C15.2, C16.2, C24.1, C4.2, C7.2, C8.2, C9.2, D7.2 (A), J3.1 (Pin_1), J3.MP (MountPin), J4.6 (VSS), J4.9 (SHIELD), R15.2, R17.2, U5.4 (GND), U7.10 (GND), U7.5 (GND)
- net CLK_OUT: now reaches R14.1, Y1.3 (OUT)
- net VDD3V3: now reaches U1.1 (VBAT)
- net VDD3V3: now also U1.19 (VDD), U1.32 (VDD), U1.48 (VDD), U1.64 (VDD), C10.1, C11.1, C12.1, C24.2, C4.1, C7.1, C8.1, C9.1, D7.1 (K), FB1.1, J3.6 (Pin_6), J4.4 (VDD), JP1.1 (A), R16.1, R18.1, U5.8 (VCC)
- net VDDA_3V3: now reaches U1.13 (VDDA)
- net VDDA_3V3: now also C15.1, C16.1, FB1.2
- net SCK: now reaches U1.21 (PA5)
- net FLASH_RST: now reaches U1.22 (PA6)
- net FLASH_RST: now also R18.2, U5.7 (~{HOLD}/~{RESET}/IO_{3})
- net WRITE_PROT: now reaches U1.23 (PA7)
- net WRITE_PROT: now also R17.1, U5.3 (~{WP}/IO_{2})
- net OCTOSPI_IO1: now reaches U1.26 (PB0)
- net OCTOSPI_IO1: now also U5.2 (DO/IO_{1})
- net OCTOSPI_IO0: now reaches U1.27 (PB1)
- net OCTOSPI_IO0: now also U5.5 (DI/IO_{0})
- net OCTOSPI_CLK: now reaches U1.28 (PB2)
- net OCTOSPI_CLK: now also U5.6 (CLK)
- net OCTOSPI_NCS: now reaches U1.29 (PB10)
- net OCTOSPI_NCS: now also R16.2, U5.1 (~{CS})
- net VCAP: now reaches U1.30 (VCAP)
- net VCAP: now also U1.62 (VCAP), C13.1, C14.1
- net USART1_TX: now reaches U1.35 (PB14)
- net GPS1_RX: now reaches U1.36 (PB15)
- net USART6_TX: now reaches U1.37 (PC6)
- net GPS2_RX: now reaches U1.38 (PC7)
- net SD_DAT0: now reaches U1.39 (PC8)
- net SD_DAT0: now also J4.7 (DAT0), U7.13 (D1-)
- net SD_DAT1: now reaches U1.40 (PC9)
- net SD_DAT1: now also J4.8 (DAT1), U7.14 (D1+)
- net RCC_MCO_OUT1: now reaches U1.41 (PA8)
- net RCC_MCO_OUT1: now also R19.2
- net GPS1_PPS: now reaches U1.42 (PA9)
- net GPS2_PPS: now reaches U1.43 (PA10)
- net SWDIO: now reaches U1.46 (PA13(JTMS)
- net SWDIO: now also J3.3 (Pin_3)
- net SWCLK: now reaches U1.49 (PA14(JTCK)
- net SWCLK: now also J3.4 (Pin_4)
- net SD_DAT2: now reaches U1.51 (PC10)
- net SD_DAT2: now also J4.1 (DAT2), U7.8 (D3-)
- net SD_DAT3: now reaches U1.52 (PC11)
- net SD_DAT3: now also J4.2 (DAT3/CD), U7.9 (D3+)
- net SD_CLK: now reaches U1.53 (PC12)
- net SD_CLK: now also J4.5 (CLK), U7.12 (D2+)
- net SD_CMD: now reaches U1.54 (PD2)
- net SD_CMD: now also J4.3 (CMD), U7.11 (D2-)
- net SWO: now reaches U1.55 (PB3(JTDO)
- net SWO: now also J3.5 (Pin_5)
- net MISO: now reaches U1.56 (PB4(NJTRST))
- net MOSI: now reaches U1.57 (PB5)
- net BOOT0: now reaches U1.60 (BOOT0)
- net BOOT0: now also JP1.2 (B), R15.1
- net NRST: now reaches U1.7 (NRST)
- net NRST: now also J3.2 (Pin_2)
- new net: R19.1, TP1.1
- no-connect marks 1 -> 7
Other:
- note added: "using the W25Q128JVSIM chip because it has QUAD IO disabled and can be optionally enabled"
- moved on the sheet: C3, R13, R14, U1, Y1
