File: carrier_board/_restore_backup_2026-09-23T15-12-00-323/carrier_board.kicad_sch (KiCad schematic)
At the start: 7 parts, among them U1 STM32H563RGTx, U2 W25Q128JVS

Commit message: 3v3
Parts:
- added D1, D2: D_Schottky, symbol Device:D_Schottky
- added J1, J2: Conn_01x02, symbol Connector_Generic:Conn_01x02
- added U3: LMR33630ADDA, Package_SO:Texas_HSOP-8-1EP_3.9x4.9mm_P1.27mm_ThermalVias, symbol Regulator_Switching:LMR33630ADDA
Connections:
- net GND: now also J1.1 (Pin_1), J2.1 (Pin_1)
- new net: D2.2 (A), J2.2 (Pin_2)
- new net: D1.1 (K), D2.1 (K), U3.2 (VIN), U3.3 (EN)
- new net: D1.2 (A), J1.2 (Pin_2)
- new net: U3.1 (GND), U3.9 (GND)
Other:
- removed sheet power
