File: carrier_board/_restore_backup_2026-09-23T17-11-02-399/carrier_board.kicad_sch (KiCad schematic)
At the start: 7 parts, among them U1 STM32H563RGTx, U2 W25Q128JVS

Commit message: 3v3
Other:
- sheet power ports: added VOUT_5V; removed VDD1_5V, VDD2_5V, VDD_RF
