File: carrier_board/carrier_board.kicad_sch (KiCad schematic)
At the start: 7 parts, among them U1 STM32H563RGTx, U2 W25Q128JVS

Commit message: im sorry
Parts:
- added U7: ZED-F9P, RF_GPS:ublox_ZED, symbol RF_GPS:ZED-F9P
- added U8: MAX-M10S, RF_GPS:ublox_MAX, symbol RF_GPS:MAX-M10S
Connections:
- new net: U7.1 (GND), U7.12 (GND), U7.14 (GND), U7.3 (GND), U7.32 (GND), U7.37 (GND), U7.41 (GND), U7.48 (GND), U7.55 (GND)
- new net: U7.33 (VCC), U7.34 (VCC)
- new net: U8.1 (GND), U8.10 (GND), U8.12 (GND)
